Commit message: Update mecanum_robot.xacro

File: src/mecanum_base/urdf/mecanum_robot.xacro (robot description, xacro)
@@ -5,12 +5,12 @@
        ========================= -->
   <!-- Geometria -->
-  <xacro:property name="wheel_radius" value="0.05"/>   <!-- Raggio ruota [m] -->
-  <xacro:property name="L" value="0.15"/>              <!-- Mezzo passo longitudinale [m] -->
-  <xacro:property name="W" value="0.15"/>              <!-- Mezzo passo trasversale [m] -->
+  <xacro:property name="wheel_radius" value="0.05"/>
+  <xacro:property name="L" value="0.15"/>
+  <xacro:property name="W" value="0.15"/>
   <!-- Hardware -->
-  <xacro:property name="mock" value="false"/>          <!-- true = simulazione, false = hardware reale -->
-  <xacro:property name="accel_limit" value="25.0"/>    <!-- Limite accelerazione [rad/s²] -->
-  <xacro:property name="ticks_per_rev" value="2048"/>  <!-- Tick encoder per giro motore -->
-  <xacro:property name="gear_ratio" value="30.0"/>     <!-- Rapporto di riduzione -->
+  <xacro:property name="mock" value="false"/>
+  <xacro:property name="accel_limit" value="25.0"/>
+  <xacro:property name="ticks_per_rev" value="2048"/>
+  <xacro:property name="gear_ratio" value="30.0"/>
   <!-- Inversione direzione ruote -->
   <xacro:property name="invert_fl" value="1"/>
@@ -21,7 +21,5 @@
        📌 LINK DI BASE
        ========================= -->
-  <!-- Link radice fittizio senza inerzia -->
   <link name="base_footprint"/>
-  <!-- Giunto fisso tra base_footprint e base_link -->
   <joint name="base_footprint_to_base_link" type="fixed">
     <parent link="base_footprint"/>
@@ -29,5 +27,4 @@
     <origin xyz="0 0 0" rpy="0 0 0"/>
   </joint>
-  <!-- Link base del robot -->
   <link name="base_link">
     <visual>
@@ -76,5 +73,5 @@
   <xacro:wheel name="rear_right_wheel"  x="${-L}" y="${-W}"/>
   <!-- =========================
-       📌 IMU (solo visualizzazione)
+       📌 IMU
        ========================= -->
   <link name="imu_link">
@@ -82,5 +79,5 @@
       <origin xyz="0 0 0" rpy="0 0 0"/>
       <geometry>
-        <box size="0.02 0.02 0.02"/> <!-- Cubo di 2 cm -->
+        <box size="0.02 0.02 0.02"/>
       </geometry>
       <material name="gray">
@@ -95,5 +92,4 @@
     </inertial>
   </link>
-  <!-- Giunto fisso tra base_link e imu_link -->
   <joint name="imu_joint" type="fixed">
     <parent link="base_link"/>
@@ -102,11 +98,52 @@
   </joint>
   <!-- =========================
-       📌 ROS2_CONTROL: HARDWARE MECANUM
+       📌 PAN/TILT CAMERA
+       ========================= -->
+  <link name="pan_link"/>
+  <joint name="pan_joint" type="revolute">
+    <parent link="base_link"/>
+    <child link="pan_link"/>
+    <origin xyz="0 0 0.15" rpy="0 0 0"/>
+    <axis xyz="0 0 1"/>
+    <limit effort="1.0" velocity="1.0" lower="-1.57" upper="1.57"/>
+  </joint>
+  <link name="tilt_link"/>
+  <joint name="tilt_joint" type="revolute">
+    <parent link="pan_link"/>
+    <child link="tilt_link"/>
+    <origin xyz="0 0 0.05" rpy="0 0 0"/>
+    <axis xyz="0 1 0"/>
+    <limit effort="1.0" velocity="1.0" lower="-1.0" upper="1.0"/>
+  </joint>
+  <!-- =========================
+       📌 SONAR VISUALI
+       ========================= -->
+  <xacro:macro name="sonar" params="name x y z">
+    <link name="${name}_link">
+      <visual>
+        <geometry>
+          <cylinder radius="0.01" length="0.02"/>
+        </geometry>
+        <origin xyz="0 0 0" rpy="1.5708 0 0"/>
+        <material name="blue">
+          <color rgba="0.2 0.2 1.0 1.0"/>
+        </material>
+      </visual>
+    </link>
+    <joint name="${name}_joint" type="fixed">
+      <parent link="base_link"/>
+      <child link="${name}_link"/>
+      <origin xyz="${x} ${y} ${z}" rpy="0 0 0"/>
+    </joint>
+  </xacro:macro>
+  <xacro:sonar name="sonar_front"  x="0.2"  y="0.0"  z="0.05"/>
+  <xacro:sonar name="sonar_left"   x="0.0"  y="0.2"  z="0.05"/>
+  <xacro:sonar name="sonar_right"  x="0.0"  y="-0.2" z="0.05"/>
+  <!-- =========================
+       📌 ROS2_CONTROL
        ========================= -->
   <ros2_control name="MecanumSystem" type="system">
     <hardware>
-      <!-- Nome del plugin hardware (corrisponde al file plugin.xml) -->
       <plugin>mecanum_hardware/MecanumSystem</plugin>
-      <!-- Parametri comuni -->
       <param name="wheel_radius">${wheel_radius}</param>
       <param name="L">${L}</param>
@@ -114,5 +151,4 @@
       <param name="mock">${mock}</param>
       <param name="accel_limit">${accel_limit}</param>
-      <!-- Parametri hardware -->
       <param name="ticks_per_rev">${ticks_per_rev}</param>
       <param name="gear_ratio">${gear_ratio}</param>
@@ -121,10 +157,8 @@
       <param name="invert_rl">${invert_rl}</param>
       <param name="invert_rr">${invert_rr}</param>
-      <!-- Parametri seriale -->
       <param name="serial_port">/dev/ttyUSB0</param>
-      <!-- <param name="baudrate">115200</param> -->
       <param name="baudrate">1000000</param>
     </hardware>
-    <!-- Interfacce per ciascun giunto -->
+    <!-- Giunti ruota -->
     <joint name="front_left_wheel_joint">
       <state_interface name="position"/>
@@ -147,4 +181,23 @@
       <command_interface name="velocity"/>
     </joint>
+    <!-- Giunti servo pan/tilt -->
+    <joint name="pan_joint">
+      <state_interface name="position"/>
+      <command_interface name="position"/>
+    </joint>
+    <joint name="tilt_joint">
+      <state_interface name="position"/>
+      <command_interface name="position"/>
+    </joint>
+    <!-- Sensori sonar -->
+    <sensor name="sonar_front">
+      <state_interface name="range"/>
+    </sensor>
+    <sensor name="sonar_left">
+      <state_interface name="range"/>
+    </sensor>
+    <sensor name="sonar_right">
+      <state_interface name="range"/>
+    </sensor>
   </ros2_control>
 </robot>

Commit message: modificato urdf file per giusto orientamento ruote e sonar

File: src/mecanum_base/urdf/mecanum_robot.xacro (robot description, xacro)
@@ -52,5 +52,6 @@
           <cylinder radius="${wheel_radius}" length="0.05"/>
         </geometry>
-        <origin xyz="0 0 0" rpy="0 0 1.5708"/>
+        <!-- ✅ Rotazione corretta sull'asse X -->
+        <origin xyz="0 0 0" rpy="1.5708 0 0"/>
         <material name="black">
           <color rgba="0.1 0.1 0.1 1.0"/>
@@ -100,5 +101,15 @@
        📌 PAN/TILT CAMERA
        ========================= -->
-  <link name="pan_link"/>
+  <link name="pan_link">
+    <visual>
+      <geometry>
+        <box size="0.03 0.03 0.01"/>
+      </geometry>
+      <origin xyz="0 0 0.005" rpy="0 0 0"/>
+      <material name="gray">
+        <color rgba="0.5 0.5 0.5 1.0"/>
+      </material>
+    </visual>
+  </link>
   <joint name="pan_joint" type="revolute">
     <parent link="base_link"/>
@@ -108,5 +119,15 @@
     <limit effort="1.0" velocity="1.0" lower="-1.57" upper="1.57"/>
   </joint>
-  <link name="tilt_link"/>
+  <link name="tilt_link">
+    <visual>
+      <geometry>
+        <box size="0.04 0.04 0.04"/>
+      </geometry>
+      <origin xyz="0 0 0.03" rpy="0 0 0"/>
+      <material name="black">
+        <color rgba="0.0 0.0 0.0 1.0"/>
+      </material>
+    </visual>
+  </link>
   <joint name="tilt_joint" type="revolute">
     <parent link="pan_link"/>
@@ -125,5 +146,6 @@
           <cylinder radius="0.01" length="0.02"/>
         </geometry>
-        <origin xyz="0 0 0" rpy="1.5708 0 0"/>
+        <!-- ✅ Ruota solo la geometria per farla puntare in avanti -->
+        <origin xyz="0 0 0" rpy="0 1.5708 0"/>
         <material name="blue">
           <color rgba="0.2 0.2 1.0 1.0"/>
@@ -134,4 +156,5 @@
       <parent link="base_link"/>
       <child link="${name}_link"/>
+      <!-- ✅ Nessuna rotazione: frame punta in avanti -->
       <origin xyz="${x} ${y} ${z}" rpy="0 0 0"/>
     </joint>
@@ -160,5 +183,5 @@
       <param name="baudrate">1000000</param>
     </hardware>
-    <!-- Giunti ruota -->
+    <!-- ✅ Interfacce di comando e stato per le ruote -->
     <joint name="front_left_wheel_joint">
       <state_interface name="position"/>
@@ -181,5 +204,5 @@
       <command_interface name="velocity"/>
     </joint>
-    <!-- Giunti servo pan/tilt -->
+    <!-- ✅ Interfacce per servo pan/tilt -->
     <joint name="pan_joint">
       <state_interface name="position"/>
@@ -190,5 +213,5 @@
       <command_interface name="position"/>
     </joint>
-    <!-- Sensori sonar -->
+    <!-- ✅ Interfacce per sensori sonar -->
     <sensor name="sonar_front">
       <state_interface name="range"/>

Commit message: Implmentato i 3 ir sensor broadcaster che ricevono dato da UART e li pubblicano su topic

File: src/mecanum_base/urdf/mecanum_robot.xacro (robot description, xacro)
@@ -100,4 +100,54 @@
     <child link="imu_link"/>
     <origin xyz="0.0 0.0 0.1" rpy="0 0 0"/>
+  </joint>
+  <!-- ========================= -->
+  <!-- Sensore IR frontale sinistro -->
+  <!-- ========================= -->
+  <link name="ir_front_left_link">
+    <!-- Visualizzazione del sensore come un piccolo cubo nero -->
+    <visual>
+      <geometry>
+        <box size="0.02 0.02 0.01"/> <!-- Dimensioni del sensore -->
+      </geometry>
+      <material name="black"/> <!-- Colore del sensore -->
+    </visual>
+  </link>
+  <!-- Joint fisso tra il sensore e il corpo del robot -->
+  <joint name="ir_front_left_joint" type="fixed">
+    <parent link="base_link"/> <!-- Collegato al corpo principale -->
+    <child link="ir_front_left_link"/> <!-- Il sensore è il figlio -->
+    <origin xyz="0.2 0.1 0.05" rpy="0 0 0"/> <!-- Posizione e orientamento -->
+  </joint>
+  <!-- ========================= -->
+  <!-- Sensore IR frontale centrale -->
+  <!-- ========================= -->
+  <link name="ir_front_center_link">
+    <visual>
+      <geometry>
+        <box size="0.02 0.02 0.01"/>
+      </geometry>
+      <material name="black"/>
+    </visual>
+  </link>
+  <joint name="ir_front_center_joint" type="fixed">
+    <parent link="base_link"/>
+    <child link="ir_front_center_link"/>
+    <origin xyz="0.2 0.0 0.05" rpy="0 0 0"/>
+  </joint>
+  <!-- ========================= -->
+  <!-- Sensore IR frontale destro -->
+  <!-- ========================= -->
+  <link name="ir_front_right_link">
+    <visual>
+      <geometry>
+        <box size="0.02 0.02 0.01"/>
+      </geometry>
+      <material name="black"/>
+    </visual>
+  </link>
+  <joint name="ir_front_right_joint" type="fixed">
+    <parent link="base_link"/>
+    <child link="ir_front_right_link"/>
+    <origin xyz="0.2 -0.1 0.05" rpy="0 0 0"/>
   </joint>
   <!-- =========================

Commit message: lettura via uart dei servo e lancio di joint broadcaster

File: src/mecanum_base/urdf/mecanum_robot.xacro (robot description, xacro)
@@ -151,4 +151,58 @@
     <origin xyz="0.2 -0.1 0.05" rpy="0 0 0"/>
   </joint>
+  <!-- Servo Pan -->
+  <joint name="servo_pan_joint" type="revolute">
+    <parent link="base_link"/>
+    <child link="servo_pan_link"/>
+    <origin xyz="0 0 0.1" rpy="0 0 0"/>
+    <axis xyz="0 0 1"/>
+    <limit effort="1.0" velocity="1.0" lower="-1.57" upper="1.57"/>
+  </joint>
+  <link name="servo_pan_link">
+    <visual>
+      <geometry>
+        <box size="0.02 0.02 0.02"/>
+      </geometry>
+      <material name="gray"/>
+    </visual>
+  </link>
+  <!-- Servo Tilt -->
+  <joint name="servo_tilt_joint" type="revolute">
+    <parent link="servo_pan_link"/>
+    <child link="servo_tilt_link"/>
+    <origin xyz="0 0 0.05" rpy="0 0 0"/>
+    <axis xyz="1 0 0"/>
+    <limit effort="1.0" velocity="1.0" lower="-1.57" upper="1.57"/>
+  </joint>
+  <link name="servo_tilt_link">
+    <visual>
+      <geometry>
+        <box size="0.02 0.02 0.02"/>
+      </geometry>
+      <material name="gray"/>
+    </visual>
+  </link>
+  <!-- 🔄 Transmission per servo_pan_joint -->
+  <transmission name="servo_pan_trans">
+    <type>transmission_interface/SimpleTransmission</type>
+    <joint name="servo_pan_joint">
+      <hardwareInterface>hardware_interface/PositionStateInterface</hardwareInterface>
+    </joint>
+    <actuator name="servo_pan_motor">
+      <hardwareInterface>hardware_interface/PositionStateInterface</hardwareInterface>
+      <mechanicalReduction>1</mechanicalReduction>
+    </actuator>
+  </transmission>
+  <!-- 🔄 Transmission per servo_tilt_joint -->
+  <transmission name="servo_tilt_trans">
+    <type>transmission_interface/SimpleTransmission</type>
+    <joint name="servo_tilt_joint">
+      <hardwareInterface>hardware_interface/PositionStateInterface</hardwareInterface>
+    </joint>
+    <actuator name="servo_tilt_motor">
+      <hardwareInterface>hardware_interface/PositionStateInterface</hardwareInterface>
+      <mechanicalReduction>1</mechanicalReduction>
+    </actuator>
+  </transmission>
   <!-- =========================
        📌 ROS2_CONTROL: HARDWARE MECANUM

Commit message: batteria broadcaster funziona. Aggiunto in git dev container

File: src/mecanum_base/urdf/mecanum_robot.xacro (robot description, xacro)
@@ -205,4 +205,23 @@
     </actuator>
   </transmission>
+  <!-- Link fittizio per la batteria -->
+  <link name="battery_link">
+    <visual>
+      <geometry>
+        <box size="0.01 0.01 0.01"/>
+      </geometry>
+      <material name="gray"/>
+    </visual>
+  </link>
+  <!-- Joint fittizio per la batteria -->
+  <joint name="battery_state" type="fixed">
+    <parent link="base_link"/> <!-- o un altro link esistente del tuo robot -->
+    <child link="battery_link"/>
+  </joint>
+  <component name="battery_monitor" type="mecanum_hardware/MecanumSystemHardware">
+  <param name="use_battery">true</param>
+  <state_interface name="voltage"/>
+  <state_interface name="percentage"/>
+  </component>
   <!-- =========================
        📌 ROS2_CONTROL: HARDWARE MECANUM

Commit message: fixed servo

File: src/mecanum_base/urdf/mecanum_robot.xacro (robot description, xacro)
@@ -5,5 +5,5 @@
        ========================= -->
   <!-- Geometria -->
-  <xacro:property name="wheel_radius" value="0.05"/>   <!-- Raggio ruota [m] -->
+  <xacro:property name="wheel_radius" value="0.025"/>   <!-- Raggio ruota [m] -->
   <xacro:property name="L" value="0.15"/>              <!-- Mezzo passo longitudinale [m] -->
   <xacro:property name="W" value="0.15"/>              <!-- Mezzo passo trasversale [m] -->
@@ -11,6 +11,6 @@
   <xacro:property name="mock" value="false"/>          <!-- true = simulazione, false = hardware reale -->
   <xacro:property name="accel_limit" value="25.0"/>    <!-- Limite accelerazione [rad/s²] -->
-  <xacro:property name="ticks_per_rev" value="2048"/>  <!-- Tick encoder per giro motore -->
-  <xacro:property name="gear_ratio" value="30.0"/>     <!-- Rapporto di riduzione -->
+  <xacro:property name="ticks_per_rev" value="12"/>  <!-- Tick encoder per giro motore -->
+  <xacro:property name="gear_ratio" value="90.0"/>     <!-- Rapporto di riduzione -->
   <!-- Inversione direzione ruote -->
   <xacro:property name="invert_fl" value="1"/>

Commit message: sistemati parametri fisici in xarco e mecanum_cmd_node

File: src/mecanum_base/urdf/mecanum_robot.xacro (robot description, xacro)
@@ -3,14 +3,19 @@
   <!-- =========================
        📌 PARAMETRI DEL ROBOT
-       ========================= -->
+       =========================
+  NOTA: // Parametri fisici dichiarati qui sono indipendenti da quelli dichiarati in mecanum_cmd_node
+       -->
   <!-- Geometria -->
-  <xacro:property name="wheel_radius" value="0.025"/>   <!-- Raggio ruota [m] -->
-  <xacro:property name="L" value="0.15"/>              <!-- Mezzo passo longitudinale [m] -->
-  <xacro:property name="W" value="0.15"/>              <!-- Mezzo passo trasversale [m] -->
+  <xacro:property name="wheel_radius" value="0.0235"/>   <!-- Raggio ruota [m] -->
+  <xacro:property name="L" value="0.7"/>              <!-- Mezzo passo longitudinale [m] -->
+  <xacro:property name="W" value="0.7"/>              <!-- Mezzo passo trasversale [m] -->
   <!-- Hardware -->
   <xacro:property name="mock" value="false"/>          <!-- true = simulazione, false = hardware reale -->
-  <xacro:property name="accel_limit" value="25.0"/>    <!-- Limite accelerazione [rad/s²] -->
+  <xacro:property name="accel_limit" value="25.0"/>     <!--Limite accelerazione [rad/s²] -->
   <xacro:property name="ticks_per_rev" value="12"/>  <!-- Tick encoder per giro motore -->
   <xacro:property name="gear_ratio" value="90.0"/>     <!-- Rapporto di riduzione -->
+  <xacro:property name="max_vx" value="0.33"/>
+  <xacro:property name="max_vy" value="0.33"/>
+  <xacro:property name="max_wz" value="4.7"/>
   <!-- Inversione direzione ruote -->
   <xacro:property name="invert_fl" value="1"/>

Commit message: sistemati parametri fisici

File: src/mecanum_base/urdf/mecanum_robot.xacro (robot description, xacro)
@@ -8,6 +8,6 @@
   <!-- Geometria -->
   <xacro:property name="wheel_radius" value="0.0235"/>   <!-- Raggio ruota [m] -->
-  <xacro:property name="L" value="0.7"/>              <!-- Mezzo passo longitudinale [m] -->
-  <xacro:property name="W" value="0.7"/>              <!-- Mezzo passo trasversale [m] -->
+  <xacro:property name="L" value="0.07"/>              <!-- Mezzo passo longitudinale [m] -->
+  <xacro:property name="W" value="0.07"/>              <!-- Mezzo passo trasversale [m] -->
   <!-- Hardware -->
   <xacro:property name="mock" value="false"/>          <!-- true = simulazione, false = hardware reale -->

Commit message: updated index

File: src/mecanum_base/urdf/mecanum_robot.xacro (robot description, xacro)
@@ -12,5 +12,5 @@
   <!-- Hardware -->
   <xacro:property name="mock" value="false"/>          <!-- true = simulazione, false = hardware reale -->
-  <xacro:property name="accel_limit" value="25.0"/>     <!--Limite accelerazione [rad/s²] -->
+  <xacro:property name="accel_limit" value="12.0"/>     <!--Limite accelerazione [rad/s²] -->
   <xacro:property name="ticks_per_rev" value="12"/>  <!-- Tick encoder per giro motore -->
   <xacro:property name="gear_ratio" value="90.0"/>     <!-- Rapporto di riduzione -->
